File: relay-replacement-board/relay-replacement-board/relay-replacement-board.kicad_pcb (KiCad board)
At the start: 2 copper layers, 100 x 50 mm, 38 parts, among them J1 Conn_01x02, J10 Conn_01x02, J11 Conn_01x02, J12 Conn_01x02, J13 Conn_01x02, J2 Conn_01x02, J3 Conn_01x02, J4 Conn_01x02, J5 Conn_01x02, J6 Conn_01x02, J7 Conn_01x02, J8 Conn_01x02, J9 Conn_01x02, Q1 NVD5865NL, Q2 NVD5865NL, Q3 NVD5865NL, Q4 NVD5865NL, Q5 NVD5865NL, Q6 NVD5865NL, Q7 NVD5865NL

Commit message: Added team logo to back silkscreen
Parts:
- added G***: LOGO, relay-replacement-board:lunar_hopper_logo_small, B.Cu at (113.0, 92.4)
